Commit message: Promote ROS 2 package to root, remove ROS 1, add Docker + CI smoke test
Finalize the ROS 2 migration:

- Remove the legacy ROS 1 (catkin) files and promote the ROS 2 package from
  ros2/omnidirectional_four_wheeled_robot/ to the repository root, giving a
  standard single-package ament_cmake layout.
- Add a reproducible Docker environment (Dockerfile + docker-entrypoint.sh)
  on ros:jazzy-ros-base with gz Harmonic, ros2_control, gz_ros2_control and
  ros_gz, building the colcon workspace.
- Add scripts/smoke_test.sh: headless functional check that launches the
  simulation (gui:=false), waits for joint_state_broadcaster /
  position_controller / velocity_controller to become active, publishes
  /cmd_vel and asserts the wheel drive joints rotate.
- Add scripts/docker_build_and_test.sh to build the image and run the smoke
  test (with optional proxy/CA wiring for restricted build networks).
- Add launch arg gui (default true) to gazebo.launch.py for headless runs.
- Add GitHub Actions workflow (.github/workflows/ci.yml) that runs the full
  build + headless smoke test on open-network runners.
- Update README for the root layout and Docker usage; update .gitignore for
  colcon.

Co-Authored-By: Claude Opus 4.8 <noreply@anthropic.com>
Claude-Session: https://claude.ai/code/session_01Gadz1scn2gzqNnkKSntfak

File: urdf/camera.urdf.xacro (robot description, xacro)
@@ -1,9 +1,9 @@
 <?xml version="1.0"?>
 <!-- ===========================================================================  -->
-<!-- |    camera.urdf.xacro																											| -->
-<!-- |    author: Koji Shibata                               										| -->
-<!-- |    e-mail: kshibata.0519@gmail.com																				| -->
-<!-- |    This is a URDF file that describes an omnidirectional 								| -->
-<!-- |    four-wheeled robot for ROS users.																			| -->
+<!-- |    camera.urdf.xacro  (ROS 2 / gz port)                                   | -->
+<!-- |    author: Koji Shibata                                                   | -->
+<!-- |    e-mail: kshibata.0519@gmail.com                                        | -->
+<!-- |    This is a URDF file that describes an omnidirectional                   | -->
+<!-- |    four-wheeled robot for ROS 2 users.                                     | -->
 <!-- ===========================================================================  -->
 <robot xmlns:xacro="http://ros.org/wiki/xacro">
@@ -15,9 +15,14 @@
 	  <origin xyz="${xyz}" rpy="${-pi/2} 0. ${-pi/2}"/>
 	</joint>
+	<!-- gz camera sensor. Handled by gz-sim-sensors-system (loaded in the    -->
+	<!-- world) and bridged to ROS via ros_gz_bridge (see config/gz_bridge.yaml). -->
 	<gazebo reference="${prefix}_link">
 	  <sensor type="camera" name="${prefix}">
-		<update_rate>30.</update_rate>
+		<always_on>1</always_on>
+		<update_rate>30</update_rate>
+		<visualize>true</visualize>
+		<topic>${prefix}/image</topic>
+		<gz_frame_id>${prefix}_link</gz_frame_id>
 		<camera name="${prefix}">
-		  <pose>0. 0. 0. 0. ${-pi/2} ${pi/2}</pose>
 		  <horizontal_fov>1.3962634</horizontal_fov>
 		  <image>
@@ -36,19 +41,4 @@
 		  </noise>
 		</camera>
-		<plugin name="camera_controller" filename="libgazebo_ros_camera.so">
-		  <alwaysOn>true</alwaysOn>
-		  <updateRate>0.</updateRate>
-		  <cameraName>/omnidirectional_four_wheeled_robot</cameraName>
-		  <cameraName>${prefix}</cameraName>
-		  <imageTopicName>image_raw</imageTopicName>
-		  <cameraInfoTopicName>camera_info</cameraInfoTopicName>
-		  <frameName>${prefix}_link</frameName>
-		  <hackBaseline>0.</hackBaseline>
-		  <distortionK1>0.</distortionK1>
-		  <distortionK2>0.</distortionK2>
-		  <distortionK3>0.</distortionK3>
-		  <distortionT1>0.</distortionT1>
-		  <distortionT2>0.</distortionT2>
-		</plugin>
 	  </sensor>
 	</gazebo>

File: urdf/laser.urdf.xacro (robot description, xacro)
@@ -1,17 +1,19 @@
 <?xml version="1.0"?>
 <!-- ===========================================================================  -->
-<!-- |    laser.urdf.xacro																											| -->
-<!-- |    author: Koji Shibata                               										| -->
-<!-- |    e-mail: kshibata.0519@gmail.com																				| -->
-<!-- |    This is a URDF file that describes an omnidirectional 								| -->
-<!-- |    four-wheeled robot for ROS users.																			| -->
+<!-- |    laser.urdf.xacro  (ROS 2 / gz port)                                    | -->
+<!-- |    author: Koji Shibata                                                   | -->
+<!-- |    e-mail: kshibata.0519@gmail.com                                        | -->
+<!-- |    This is a URDF file that describes an omnidirectional                   | -->
+<!-- |    four-wheeled robot for ROS 2 users.                                     | -->
 <!-- ===========================================================================  -->
 <robot xmlns:xacro="http://ros.org/wiki/xacro">
 	<xacro:macro name="laser_macro" params="parent prefix xyz rpy">
 		<link name="${prefix}_link">
+			<!-- The original Hokuyo .dae mesh is not shipped with gz, so a small  -->
+			<!-- box placeholder is used for visual/collision.                     -->
 			<collision>
 				<origin xyz="0. 0. 0." rpy="0. 0. 0."/>
 				<geometry>
-					<mesh filename="package://gazebo_plugins/test/multi_robot_scenario/meshes/laser/hokuyo.dae"/>
+					<box size="0.05 0.05 0.07"/>
 				</geometry>
 			</collision>
@@ -19,6 +21,9 @@
 				<origin xyz="0. 0. 0." rpy="0. 0. 0."/>
 				<geometry>
-					<mesh filename="package://gazebo_plugins/test/multi_robot_scenario/meshes/laser/hokuyo.dae"/>
+					<box size="0.05 0.05 0.07"/>
 				</geometry>
+				<material name="Gray">
+					<color rgba="0.5 0.5 0.5 1."/>
+				</material>
 			</visual>
 			<inertial>
@@ -33,15 +38,19 @@
 			<child link="${prefix}_link"/>
 		</joint>
-		<!-- Hokuyo sensor for simulation -->
+		<!-- gz GPU lidar. Handled by gz-sim-sensors-system and bridged to ROS    -->
+		<!-- (sensor_msgs/LaserScan) via ros_gz_bridge.                           -->
 		<gazebo reference="${prefix}_link">
-			<sensor type="ray" name="${prefix}_sensor">
+			<sensor type="gpu_lidar" name="${prefix}_sensor">
 				<pose>0. 0. 0. 0. 0. 0.</pose>
+				<always_on>1</always_on>
 				<visualize>true</visualize>
-				<update_rate>40.</update_rate>
-				<ray>
+				<update_rate>40</update_rate>
+				<topic>${prefix}/scan</topic>
+				<gz_frame_id>${prefix}_link</gz_frame_id>
+				<lidar>
 					<scan>
 						<horizontal>
 							<samples>1080</samples>
-							<resolution>0.25</resolution>
+							<resolution>1</resolution>
 							<min_angle>${-3*pi/4}</min_angle>
 							<max_angle>${3*pi/4}</max_angle>
@@ -51,20 +60,12 @@
 						<min>0.1</min>
 						<max>30.</max>
-						<resolution>1.e-3</resolution>
+						<resolution>0.01</resolution>
 					</range>
 					<noise>
-						<!-- Noise parameters based on published spec for Hokuyo laser 			-->
-						<!-- achieving "+-30mm" accuracy at range < 10m.  A mean of 0.0m and 		-->
-						<!-- stddev of 0.01m will put 99.7% of samples within 0.03m of the true 	-->
-						<!-- reading. 																	-->
 						<type>gaussian</type>
 						<mean>0.</mean>
 						<stddev>1.e-3</stddev>
 					</noise>
-				</ray>
-				<plugin name="gazebo_ros_head_hokuyo_controller" filename="libgazebo_ros_laser.so">
-					<topicName>/omnidirectional_four_wheeled_robot/${prefix}_scan</topicName>
-					<frameName>${prefix}_link</frameName>
-				</plugin>
+				</lidar>
 			</sensor>
 		</gazebo>

File: urdf/robot.urdf.xacro (robot description, xacro)
@@ -1,11 +1,11 @@
 <?xml version="1.0"?>
 <!-- ===========================================================================  -->
-<!-- |    ommidirecctional_four-wheeled_robot.urdf.xacro												| -->
-<!-- |    author: Koji Shibata                               										| -->
-<!-- |    e-mail: kshibata.0519@gmail.com																				| -->
-<!-- |    This is a URDF file that describes an omnidirectional 								| -->
-<!-- |    four-wheeled robot for ROS users.																			| -->
+<!-- |    robot.urdf.xacro  (ROS 2 / gz port)                                    | -->
+<!-- |    author: Koji Shibata                                                   | -->
+<!-- |    e-mail: kshibata.0519@gmail.com                                        | -->
+<!-- |    This is a URDF file that describes an omnidirectional                   | -->
+<!-- |    four-wheeled robot for ROS 2 users.                                     | -->
 <!-- ===========================================================================  -->
-<robot name="omnidirectional_four-wheeled_robot" xmlns:xacro="http://ros.org/wiki/xacro">
+<robot name="omnidirectional_four_wheeled_robot" xmlns:xacro="http://ros.org/wiki/xacro">
 <xacro:property name="x_size" value="0.75"/>
 <xacro:property name="y_size" value="0.75"/>
@@ -17,8 +17,10 @@
 <xacro:property name="effort_limit" value="1."/>
 <xacro:property name="velocity_limit" value="5."/>
-<xacro:property name="control_period" value="0.001"/>
-<xacro:include filename="$(find omnidirectional_four-wheeled_robot)/urdf/wheel.urdf.xacro"/>
-<xacro:include filename="$(find omnidirectional_four-wheeled_robot)/urdf/camera.urdf.xacro"/>
-<xacro:include filename="$(find omnidirectional_four-wheeled_robot)/urdf/laser.urdf.xacro"/>
+<!-- Absolute path to the ros2_control controller configuration.                -->
+<!-- Passed in from the launch file (resolved from the package share dir).      -->
+<xacro:arg name="controllers_config" default=""/>
+<xacro:include filename="$(find omnidirectional_four_wheeled_robot)/urdf/wheel.urdf.xacro"/>
+<xacro:include filename="$(find omnidirectional_four_wheeled_robot)/urdf/camera.urdf.xacro"/>
+<xacro:include filename="$(find omnidirectional_four_wheeled_robot)/urdf/laser.urdf.xacro"/>
 	<link name="base_link"/>
 	<link name="body_link">
@@ -60,6 +62,6 @@
 		<inertial>
 			<origin xyz="0. 0. 0."/>
-			<mass value="0."/>
-			<inertia ixx="0." ixy="0." ixz="0." iyy="0." iyz="0." izz="0."/>
+			<mass value="1.e-6"/>
+			<inertia ixx="1.e-6" ixy="0." ixz="0." iyy="1.e-6" iyz="0." izz="1.e-6"/>
 		</inertial>
 	</link>
@@ -68,5 +70,4 @@
 		<parent link="base_link"/>
 		<child link="body_link"/>
-		<calibration rising="0."/>
 		<dynamics damping="0." friction="0."/>
 	</joint>
@@ -83,28 +84,47 @@
 	<!-- <xacro:laser_macro prefix="FrontLaser" parent="body_link" xyz="${x_size/4} 0. ${z_size/2 + 1.e-2}" rpy="0. 0. 0."/>
 	<xacro:laser_macro prefix="RearLaser" parent="body_link" xyz="${-x_size/4} 0. ${z_size/2 + 1.e-2}" rpy="0. 0. ${-pi}"/> -->
+	<!-- ros2_control: a single system aggregating all 8 wheel joints. -->
+	<ros2_control name="GazeboSimSystem" type="system">
+		<hardware>
+			<plugin>gz_ros2_control/GazeboSimSystem</plugin>
+		</hardware>
+		<xacro:wheel_ros2_control suffix="FRwheel"/>
+		<xacro:wheel_ros2_control suffix="RRwheel"/>
+		<xacro:wheel_ros2_control suffix="FLwheel"/>
+		<xacro:wheel_ros2_control suffix="RLwheel"/>
+	</ros2_control>
 	<gazebo reference="base_link">
-		<selfCollide>false</selfCollide>
 		<mu1 value="0.05"/>
 		<mu2 value="0.05"/>
 	</gazebo>
 	<gazebo reference="frontPoint_link">
-		<selfCollide>false</selfCollide>
 		<material>Gazebo/Red</material>
 	</gazebo>
+	<!-- IMU sensor (handled by gz-sim-imu-system, bridged to ROS). -->
+	<gazebo reference="body_link">
+		<sensor name="imu_sensor" type="imu">
+			<always_on>1</always_on>
+			<update_rate>50</update_rate>
+			<topic>imu</topic>
+			<gz_frame_id>body_link</gz_frame_id>
+			<imu>
+				<angular_velocity>
+					<x><noise type="gaussian"><mean>0.</mean><stddev>1.e-3</stddev></noise></x>
+					<y><noise type="gaussian"><mean>0.</mean><stddev>1.e-3</stddev></noise></y>
+					<z><noise type="gaussian"><mean>0.</mean><stddev>1.e-3</stddev></noise></z>
+				</angular_velocity>
+				<linear_acceleration>
+					<x><noise type="gaussian"><mean>0.</mean><stddev>1.e-3</stddev></noise></x>
+					<y><noise type="gaussian"><mean>0.</mean><stddev>1.e-3</stddev></noise></y>
+					<z><noise type="gaussian"><mean>0.</mean><stddev>1.e-3</stddev></noise></z>
+				</linear_acceleration>
+			</imu>
+		</sensor>
+	</gazebo>
+	<!-- gz_ros2_control system plugin: loads the controller_manager inside gz. -->
 	<gazebo>
-		<plugin name="gazebo_ros_control" filename="libgazebo_ros_control.so">
-			<controlPeriod>${control_period}</controlPeriod>
-			<legacyModeNS>true</legacyModeNS>
-			<robotParam>/robot_description</robotParam>
-			<robotNamespace>/omnidirectional_four_wheeled_robot</robotNamespace>
-			<robotSimType>gazebo_ros_control/DefaultRobotHWSim</robotSimType>
-		</plugin>
-		<plugin name="imu_plugin" filename="libgazebo_ros_imu.so">
-			<alwaysOn>true</alwaysOn>
-			<bodyName>body_link</bodyName>
-			<topicName>/omnidirectional_four_wheeled_robot/imu</topicName>
-			<serviceName>imu_service</serviceName>
-			<gaussianNoise>1.e-3</gaussianNoise>
-			<updateRate>50.</updateRate>
+		<plugin filename="gz_ros2_control-system"
+				name="gz_ros2_control::GazeboSimROS2ControlPlugin">
+			<parameters>$(arg controllers_config)</parameters>
 		</plugin>
 	</gazebo>

File: urdf/wheel.urdf.xacro (robot description, xacro)
@@ -1,11 +1,12 @@
 <?xml version="1.0"?>
 <!-- ===========================================================================  -->
-<!-- |    wheel.urdf.xacro																											| -->
-<!-- |    author: Koji Shibata                               										| -->
-<!-- |    e-mail: kshibata.0519@gmail.com																				| -->
-<!-- |    This is a URDF file that describes an omnidirectional 								| -->
-<!-- |    four-wheeled robot for ROS users.																			| -->
+<!-- |    wheel.urdf.xacro  (ROS 2 / gz port)                                    | -->
+<!-- |    author: Koji Shibata                                                   | -->
+<!-- |    e-mail: kshibata.0519@gmail.com                                        | -->
+<!-- |    This is a URDF file that describes an omnidirectional                   | -->
+<!-- |    four-wheeled robot for ROS 2 users.                                     | -->
 <!-- ===========================================================================  -->
 <robot xmlns:xacro="http://ros.org/wiki/xacro">
+	<!-- Kinematic/visual description of one wheel (steering link + drive link). -->
 	<xacro:macro name="wheel_macro" params="suffix parent x_pos y_pos">
 		<link name="${suffix}_link1">
@@ -57,4 +58,5 @@
 			</inertial>
 		</link>
+		<!-- joint1: steering (position controlled) -->
 		<joint name="${suffix}_joint1" type="continuous">
 			<origin xyz="${x_pos} ${y_pos} 0." rpy="0. 0. 0."/>
@@ -62,7 +64,7 @@
 			<parent link="${parent}"/>
 			<child link="${suffix}_link1"/>
-			<calibration rising="0."/>
 			<dynamics damping="1." friction="0."/>
 		</joint>
+		<!-- joint2: drive (velocity controlled) -->
 		<joint name="${suffix}_joint2" type="continuous">
 			<origin xyz="0. 0. 0." rpy="0. 0. 0."/>
@@ -70,29 +72,7 @@
 			<parent link="${suffix}_link1"/>
 			<child link="${suffix}_link2"/>
-			<calibration rising="0."/>
 			<dynamics damping="1." friction="0."/>
 		</joint>
-		<transmission name="${suffix}_trans1">
-			<type>transmission_interface/SimpleTransmission</type>
-			<joint name="${suffix}_joint1">
-				<hardwareInterface>hardware_interface/PositionJointInterface</hardwareInterface>
-			</joint>
-			<actuator name="${suffix}_motor1">
-				<mechanicalReduction>1</mechanicalReduction>
-				<hardwareInterface>hardware_interface/PositionJointInterface</hardwareInterface>
-			</actuator>
-		</transmission>
-		<transmission name="${suffix}_trans2">
-			<type>transmission_interface/SimpleTransmission</type>
-			<joint name="${suffix}_joint2">
-				<hardwareInterface>hardware_interface/VelocityJointInterface</hardwareInterface>
-			</joint>
-			<actuator name="${suffix}_motor2">
-				<mechanicalReduction>1</mechanicalReduction>
-				<hardwareInterface>hardware_interface/VelocityJointInterface</hardwareInterface>
-			</actuator>
-		</transmission>
 		<gazebo reference="${suffix}_link1">
-			<selfCollide>false</selfCollide>
 			<mu1 value="0.05"/>
 			<mu2 value="0.05"/>
@@ -100,5 +80,4 @@
 		</gazebo>
 		<gazebo reference="${suffix}_link2">
-			<selfCollide>false</selfCollide>
 			<mu1 value="0.80"/>
 			<mu2 value="0.80"/>
@@ -106,3 +85,24 @@
 		</gazebo>
 	</xacro:macro>
+	<!-- ros2_control joint entries for one wheel.                                -->
+	<!-- joint1 = steering (position command), joint2 = drive (velocity command). -->
+	<!-- Call this inside a single <ros2_control> block in robot.urdf.xacro.      -->
+	<xacro:macro name="wheel_ros2_control" params="suffix">
+		<joint name="${suffix}_joint1">
+			<command_interface name="position">
+				<param name="min">-${pi}</param>
+				<param name="max">${pi}</param>
+			</command_interface>
+			<state_interface name="position"/>
+			<state_interface name="velocity"/>
+		</joint>
+		<joint name="${suffix}_joint2">
+			<command_interface name="velocity">
+				<param name="min">-${velocity_limit}</param>
+				<param name="max">${velocity_limit}</param>
+			</command_interface>
+			<state_interface name="position"/>
+			<state_interface name="velocity"/>
+		</joint>
+	</xacro:macro>
 </robot>
